Commit message: Add ergoCub2 arm

File: urdf/ergoCub/robots/ergoCubGazeboV1/model.urdf (robot description, URDF)
Before this commit: robot ergoCub, 194 links, 193 joints
Links:
- added link l_elbow_m, mass 0.8; collision sphere radius=0.03; visual sphere radius=0.03
- added link r_elbow_m, mass 0.8; collision sphere radius=0.03; visual sphere radius=0.03
- link l_shoulder_2: mass 0.440933 -> 1.1
- link l_shoulder_3: mass 0.271466 -> 0.33
- link l_upperarm: mass 1.77085 -> 0.91; geometry 
- link r_shoulder_2: mass 0.439227 -> 1.1
- link r_shoulder_3: mass 0.271466 -> 0.33
- link r_upperarm: mass 1.77224 -> 0.91; geometry 
Joints:
- added joint l_elbow_m: type fixed, parent l_forearm, child l_elbow_m, origin xyz=0 0 0 rpy=0 0 0, axis 0 0 0
- added joint r_elbow_m: type fixed, parent r_forearm, child r_elbow_m, origin xyz=0 0 0 rpy=0 0 0, axis 0 0 0
- joint l_arm_ft_sensor: origin xyz=-0.004350065786786487 2.435985168580679e-07 -0.054299880148590496 rpy=0 0 0 -> xyz=-0.016 0.0 -0.0807 rpy=0 0 0
- joint l_elbow: origin xyz=0.01000011478523053 -0.001500064220488484 -0.12369962531821438 rpy=0 0 0 -> xyz=0.010 0.0 -0.0519 rpy=0 0 0
- joint l_shoulder_yaw: origin xyz=0 0 -0.022500225580001282 rpy=0 0 0 -> xyz=0.0 0.0 -0.0689 rpy=0 0 0
- joint l_wrist_yaw: origin xyz=-0.015000090840254894 0.0020007008753266664 -0.19435007309759766 rpy=0 0 0 -> xyz=-0.012 0.0 -0.22835 rpy=0 0 0
- joint r_arm_ft_sensor: origin xyz=-0.006849910543190453 3.2679315392636354e-07 -0.05429971877536288 rpy=0 0 0 -> xyz=-0.016 0.0 -0.0807 rpy=0 0 0
- joint r_elbow: origin xyz=0.010000044612835832 0.0015000724494400042 -0.1236996308912752 rpy=0 0 0 -> xyz=0.010 0.0 -0.0519 rpy=0 0 0
- joint r_shoulder_yaw: origin xyz=0 0 -0.02250022557998886 rpy=0 0 0 -> xyz=0.0 0.0 -0.0689 rpy=0 0 0
- joint r_wrist_yaw: origin xyz=-0.015000200282364597 -0.002000693647607188 -0.19435006472514327 rpy=0 0 0 -> xyz=-0.012 0.0 -0.22835 rpy=0 0 0

File: urdf/ergoCub/robots/ergoCubSN000/model.urdf (robot description, URDF)
Before this commit: robot ergoCub, 194 links, 193 joints
Links:
- added link l_elbow_m, mass 0.8; collision sphere radius=0.03; visual sphere radius=0.03
- added link r_elbow_m, mass 0.8; collision sphere radius=0.03; visual sphere radius=0.03
- link l_shoulder_2: mass 0.440933 -> 1.1
- link l_shoulder_3: mass 0.271466 -> 0.33
- link l_upperarm: mass 1.77085 -> 0.91; geometry 
- link r_shoulder_2: mass 0.439227 -> 1.1
- link r_shoulder_3: mass 0.271466 -> 0.33
- link r_upperarm: mass 1.77224 -> 0.91; geometry 
Joints:
- added joint l_elbow_m: type fixed, parent l_forearm, child l_elbow_m, origin xyz=0 0 0 rpy=0 0 0, axis 0 0 0
- added joint r_elbow_m: type fixed, parent r_forearm, child r_elbow_m, origin xyz=0 0 0 rpy=0 0 0, axis 0 0 0
- joint l_arm_ft_sensor: origin xyz=-0.004350065786786487 2.435985168580679e-07 -0.054299880148590496 rpy=0 0 0 -> xyz=-0.016 0.0 -0.0807 rpy=0 0 0
- joint l_elbow: origin xyz=0.01000011478523053 -0.001500064220488484 -0.12369962531821438 rpy=0 0 0 -> xyz=0.010 0.0 -0.0519 rpy=0 0 0
- joint l_shoulder_yaw: origin xyz=0 0 -0.022500225580001282 rpy=0 0 0 -> xyz=0.0 0.0 -0.0689 rpy=0 0 0
- joint l_wrist_yaw: origin xyz=-0.015000090840254894 0.0020007008753266664 -0.19435007309759766 rpy=0 0 0 -> xyz=-0.012 0.0 -0.22835 rpy=0 0 0
- joint r_arm_ft_sensor: origin xyz=-0.006849910543190453 3.2679315392636354e-07 -0.05429971877536288 rpy=0 0 0 -> xyz=-0.016 0.0 -0.0807 rpy=0 0 0
- joint r_elbow: origin xyz=0.010000044612835832 0.0015000724494400042 -0.1236996308912752 rpy=0 0 0 -> xyz=0.010 0.0 -0.0519 rpy=0 0 0
- joint r_shoulder_yaw: origin xyz=0 0 -0.02250022557998886 rpy=0 0 0 -> xyz=0.0 0.0 -0.0689 rpy=0 0 0
- joint r_wrist_yaw: origin xyz=-0.015000200282364597 -0.002000693647607188 -0.19435006472514327 rpy=0 0 0 -> xyz=-0.012 0.0 -0.22835 rpy=0 0 0
